File: psu.sch (KiCad schematic (older format))
At the start: 63 parts, among them J1 Screw_Terminal_01x02, J2 Barrel_Jack, J3 Binding posts, SW1 SW_SP4T, SW2 SW_SP4T, SW3 Lever toggle, U1 LM4040DBZ-2.5, U2 LT3081, U3 LM393, U4 LM334M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

Commit message: Rev B
Other:
- note added: "Alex Striff <striffa@reed.edu> <https://github.com/jfjhh/lab-psu>"
- note added: "B"
- note added: "These inputs are backwards.\nOn the PCB, the traces should be cut\nand wires used to switch the inputs."
- note removed: "A"
Changed lines of the file:
@@
 $EndDescr
 Text Notes 10600 7650 0    50   ~ 0
-A
+B
 Text Notes 8150 7650 0    50   ~ 0
 2019-06-01
@@
 	0    1    1    0
 $EndComp
+Wire Notes Line
+	6000 6100 6000 6500
+Text Notes 5350 6750 0    50   Italic 0
+These inputs are backwards.\nOn the PCB, the traces should be cut\nand wires used to switch the inputs.
+Text Notes 8550 7500 0    50   ~ 0
+Alex Striff <striffa@reed.edu> <https://github.com/jfjhh/lab-psu>
 $EndSCHEMATC
